File: KiCad/PCB_V1/PCB_V1.kicad_sch (KiCad schematic)
At the start: 0 parts

Commit message: gyro+ble schematic
Parts:
- added C1, C2, C3: 100nF, Capacitor_SMD:C_0805_2012Metric_Pad1.18x1.45mm_HandSolder, symbol Device:C
- added C4: 100nF, symbol Device:C
- added D1: PESD3V3U1UL, lcsc_footprints:C19829543_SOD-882_L1_0-W0_6-RD, symbol lcsc_imported:PESD3V3U1UL
- added J1: Conn_01x06_Socket, Connector_PinSocket_2.54mm:PinSocket_1x06_P2.54mm_Vertical, symbol Connector:Conn_01x06_Socket
- added U1: MT6701CT-ACD_C50203010, lcsc_footprints:C50203010_SOIC-8_L5_0-W4_0-P1_27-LS6_0-BL, symbol lcsc_imported:MT6701CT-ACD_C50203010
- added U2: STM32F411RET6, lcsc_footprints:C94355_LQFP-64_L10_0-W10_0-P0_50-LS12_0-BL, symbol lcsc_imported:STM32F411RET6
- added U3: LSM6DSOXTR, lcsc_footprints:C481766_LGA-14L_L3_0-W2_5-P0_50-TL, symbol lcsc_imported:LSM6DSOXTR
Connections:
- new net +3V3: C1.1, C2.1, C3.1, C4.2, D1.1 (K), J1.5 (Pin_5), U1.1 (VDD), U3.5 (VDDIO), U3.8 (VDD)
- new net GND: C1.2, C2.2, C3.2, C4.1, D1.2 (A), J1.4 (Pin_4), U1.2 (MODE), U1.4 (GND), U3.2 (SDX), U3.3 (SCX), U3.6 (GND), U3.7 (GND)
- new net HC-05 STATE: J1.1 (Pin_1), U2.41 (PA8)
- new net SPI2_CS: U2.33 (PB12), U3.12 (CS)
- new net SPI2_MISO: U2.35 (PB14), U3.1 (SDO/SA0)
- new net SPI2_MOSI: U2.36 (PB15), U3.14 (SDA)
- new net SPI2_SCK: U2.34 (PB13), U3.13 (SCL)
- new net USART1_RX: J1.3 (Pin_3), U2.43 (PA10)
- new net USART1_TX: J1.2 (Pin_2), U2.42 (PA9)
- no-connect marks 0 -> 8
Other:
- note added: "Gyro"
- note added: "HC-05 connector"
- title: (none) -> Schematic

Commit message: buck+LDO schematic
Parts:
- added C10, C11: 1uF, lcsc_footprints:C5250745_SOT-563-6_L1_6-W1_2-P0_50-LS1_6-BL, symbol Device:C
- added C5: 10uF, lcsc_footprints:C5250745_SOT-563-6_L1_6-W1_2-P0_50-LS1_6-BL, symbol Device:C
- added C6: 330nF, symbol Device:C
- added C7: 100pF, lcsc_footprints:C5349667_IND-SMD_L4_4-W4_2, symbol Device:C
- added C8, C9: 22uF, lcsc_footprints:C5250745_SOT-563-6_L1_6-W1_2-P0_50-LS1_6-BL, symbol Device:C
- added L1: APH0420T3R3M, lcsc_footprints:C5349667_IND-SMD_L4_4-W4_2, symbol lcsc_imported:APH0420T3R3M
- added R1: 52.3k, Resistor_SMD:R_0805_2012Metric_Pad1.20x1.40mm_HandSolder, symbol Device:R
- added R2: 10k, symbol Device:R
- added U4: AP62300Z6-7, lcsc_footprints:C5250745_SOT-563-6_L1_6-W1_2-P0_50-LS1_6-BL, symbol lcsc_imported:AP62300Z6-7
- added U5: TLV75533PDBVR, lcsc_footprints:C404027_SOT-23-5_L3_0-W1_7-P0_95-LS2_8-BR, symbol lcsc_imported:TLV75533PDBVR
Connections:
- net +3V3: now also C11.1, U5.5 (OUT)
- net GND: now also C10.2, C11.2, C5.2, C8.2, C9.2, R2.2, U4.3 (GND), U5.2 (GND)
- new net: C7.2, R1.2, R2.1, U4.6 (FB)
- new net: C6.2, L1.1, U4.2 (SW)
- new net: C6.1, U4.4 (BST)
- new net +5V: C10.1, C7.1, C8.1, C9.1, L1.2, R1.1, U4.5 (EN), U5.1 (IN), U5.3 (EN)
- new net +BATT: C5.1, U4.1 (VIN)
- no-connect marks 8 -> 9
Other:
- note added: "Buck source"
- note added: "LDO 3v3"
- note added: "Notes: -change to BD9G101G and power the motors directly from the battery. No need for the 3A that i have now -design reverse polarity protection (order TVS(?) diode)"

Commit message: LCSC lib moved + uC minimal
Parts:
- removed C11: 1uF, lcsc_footprints:C5250745_SOT-563-6_L1_6-W1_2-P0_50-LS1_6-BL, symbol Device:C
- removed D1: PESD3V3U1UL, lcsc_footprints:C19829543_SOD-882_L1_0-W0_6-RD, symbol lcsc_imported:PESD3V3U1UL
- removed L1: APH0420T3R3M, lcsc_footprints:C5349667_IND-SMD_L4_4-W4_2, symbol lcsc_imported:APH0420T3R3M
- removed U1: MT6701CT-ACD_C50203010, lcsc_footprints:C50203010_SOIC-8_L5_0-W4_0-P1_27-LS6_0-BL, symbol lcsc_imported:MT6701CT-ACD_C50203010
- removed U2: STM32F411RET6, lcsc_footprints:C94355_LQFP-64_L10_0-W10_0-P0_50-LS12_0-BL, symbol lcsc_imported:STM32F411RET6
- removed U3: LSM6DSOXTR, lcsc_footprints:C481766_LGA-14L_L3_0-W2_5-P0_50-TL, symbol lcsc_imported:LSM6DSOXTR
- removed U4: AP62300Z6-7, lcsc_footprints:C5250745_SOT-563-6_L1_6-W1_2-P0_50-LS1_6-BL, symbol lcsc_imported:AP62300Z6-7
- removed U5: TLV75533PDBVR, lcsc_footprints:C404027_SOT-23-5_L3_0-W1_7-P0_95-LS2_8-BR, symbol lcsc_imported:TLV75533PDBVR
- added C13, C25, C29, C31, C33, C35: 4.7uF, LCSC:C_0805_2012Metric_Pad1.18x1.45mm_HandSolder, symbol Device:C
- added C16, C18, C30: 1uF, LCSC:C_0805_2012Metric_Pad1.18x1.45mm_HandSolder, symbol Device:C
- added C19: 47uF, LCSC:C_0805_2012Metric_Pad1.18x1.45mm_HandSolder, symbol Device:C
- added C22, C26, C27, C28, C32, C34, C36: 100nF, LCSC:C_0805_2012Metric_Pad1.18x1.45mm_HandSolder, symbol Device:C
- added C23, C24: 33pF, LCSC:C_0805_2012Metric_Pad1.18x1.45mm_HandSolder, symbol Device:C
- added D1, D4: PESD3V3U1UL, LCSC:C19829543_SOD-882_L1_0-W0_6-RD, symbol LCSC:PESD3V3U1UL
- added D2: SS16-E3/61T, LCSC:C183023_SMA_L4_3-W2_6-LS5_2-RD, symbol LCSC:SS16-E3/61T
- added D3: SMAJ33A, LCSC:C223988_SMA_L4_3-W2_6-LS5_0-RD, symbol LCSC:SMAJ33A_C223988
- added J2: Conn_01x02_Pin, Connector_PinHeader_2.54mm:PinHeader_1x02_P2.54mm_Vertical, symbol Connector:Conn_01x02_Pin
- added J3: Conn_01x07_Pin, Connector_PinHeader_2.54mm:PinHeader_1x07_P2.54mm_Vertical, symbol Connector:Conn_01x07_Pin
- added L1: APH0420T3R3M, LCSC:C5349667_IND-SMD_L4_4-W4_2, symbol LCSC:APH0420T3R3M
- added LED4: XL-2012UGC, LCSC:C965815_LED0805-RD_GREEN, symbol LCSC:XL-2012UGC
- added R15: 0, LCSC:R_0805_2012Metric_Pad1.20x1.40mm_HandSolder, symbol Device:R
- added R16: 100, LCSC:R_0805_2012Metric_Pad1.20x1.40mm_HandSolder, symbol Device:R
- added R17: 4.7k, LCSC:R_0805_2012Metric_Pad1.20x1.40mm_HandSolder, symbol Device:R
- added R18: 10k, LCSC:R_0805_2012Metric_Pad1.20x1.40mm_HandSolder, symbol Device:R
- added R21: 330 Ohm, LCSC:R_0805_2012Metric_Pad1.20x1.40mm_HandSolder, symbol Device:R
- added R8: 10 Ohm, LCSC:R_0805_2012Metric_Pad1.20x1.40mm_HandSolder, symbol Device:R
- added SW1, SW2: TS60110-411-03015, LCSC:C42400889_SW-SMD_4P-L5_2-W5_2-P3_70-LS6_4-BL, symbol LCSC:TS60110-411-03015
- added U1: LSM6DSOXTR, LCSC:C481766_LGA-14L_L3_0-W2_5-P0_50-TL, symbol LCSC:LSM6DSOXTR
- added U2, U6: MT6701CT-ACD_C50203010, LCSC:C50203010_SOIC-8_L5_0-W4_0-P1_27-LS6_0-BL, symbol LCSC:MT6701CT-ACD_C50203010
- added U3: STM32F411RET6, LCSC:C94355_LQFP-64_L10_0-W10_0-P0_50-LS12_0-BL, symbol LCSC:STM32F411RET6
- added U4: AP62300Z6-7, LCSC:C5250745_SOT-563-6_L1_6-W1_2-P0_50-LS1_6-BL, symbol LCSC:AP62300Z6-7
- added U5: TLV75533PDBVR, LCSC:C404027_SOT-23-5_L3_0-W1_7-P0_95-LS2_8-BR, symbol LCSC:TLV75533PDBVR
- added X1: X49SS2-8.000-F20JGDT, LCSC:C2842263_CRYSTAL-SMD_L11_4-W4_7-LS12_7, symbol LCSC:X49SS2-8_000-F20JGDT
- C1, C2, C3: footprint Capacitor_SMD:C_0805_2012Metric_Pad1.18x1.45mm_HandSolder -> LCSC:C_0805_2012Metric_Pad1.18x1.45mm_HandSolder
- C10: value 1uF -> 100nF; footprint lcsc_footprints:C5250745_SOT-563-6_L1_6-W1_2-P0_50-LS1_6-BL -> LCSC:C_0805_2012Metric_Pad1.18x1.45mm_HandSolder
- C4, C6: footprint (none) -> LCSC:C_0805_2012Metric_Pad1.18x1.45mm_HandSolder
- C5, C8, C9: footprint lcsc_footprints:C5250745_SOT-563-6_L1_6-W1_2-P0_50-LS1_6-BL -> LCSC:C_0805_2012Metric_Pad1.18x1.45mm_HandSolder
- C7: footprint lcsc_footprints:C5349667_IND-SMD_L4_4-W4_2 -> LCSC:C_0805_2012Metric_Pad1.18x1.45mm_HandSolder
- R1: footprint Resistor_SMD:R_0805_2012Metric_Pad1.20x1.40mm_HandSolder -> LCSC:R_0805_2012Metric_Pad1.20x1.40mm_HandSolder
- R2: footprint (none) -> LCSC:R_0805_2012Metric_Pad1.20x1.40mm_HandSolder
Connections:
- net +3V3: now also C10.1, C18.1, C25.1, C26.1, C31.1, C32.1, C33.1, C34.1, C35.1, C36.1, D1.1 (K), D4.1 (K), J3.7 (Pin_7), R17.2, R8.1, U1.5 (VDDIO), U1.8 (VDD), U2.1 (VDD), U3.1 (VBAT), U3.19 (VDD), U3.32 (VDD), U3.48 (VDD), U3.64 (VDD), U5.5 (OUT), U6.1 (VDD)
- net +5V: now also C16.1, L1.2, R21.2, U4.5 (EN), U5.1 (IN), U5.3 (EN); no longer C10.1
- net +BATT: now also C13.1, D2.1 (C), D3.1 (K), U4.1 (VIN)
- net GND: now also C13.2, C16.2, C18.2, C19.2, C22.2, C23.2, C24.2, C25.2, C26.2, C27.2, C29.2, C30.2, C31.2, C32.2, C33.2, C34.2, C35.2, C36.2, D1.2 (A), D3.2 (A), D4.2 (A), J2.2 (Pin_2), J3.4 (Pin_4), LED4.1 (K), R16.1, R18.2, SW1.1, SW1.2, SW2.3, SW2.4, U1.2 (SDX), U1.3 (SCX), U1.7 (GND), U2.2 (MODE), U2.4 (GND), U3.12 (VSSA/VREF-), U3.18 (VSS), U3.31 (VSS), U3.47 (VSS), U3.63 (VSS), U4.3 (GND), U5.2 (GND), U6.2 (MODE), U6.4 (GND)
- net HC-05 STATE: now also U3.41 (PA8)
- net SPI2_CS: now also U1.12 (CS), U3.33 (PB12)
- net SPI2_MISO: now also U1.1 (SDO/SA0), U3.35 (PB14)
- net SPI2_MOSI: now also U1.14 (SDA), U3.36 (PB15)
- net SPI2_SCK: now also U1.13 (SCL), U3.34 (PB13)
- net USART1_RX: now also U3.43 (PA10)
- net USART1_TX: now also U3.42 (PA9)
- net at C7.2, R1.2, R2.1: now also U4.6 (FB)
- net at C6.2: now also L1.1, U4.2 (SW)
- net at C6.1: now also U4.4 (BST)
- new net: R18.1, U3.60 (BOOT0)
- new net: C24.1, R15.1, X1.2 (OSC2)
- new net: D2.2 (A), J2.1 (Pin_1)
- new net: C28.1, R17.1, SW2.1, SW2.2
- new net: LED4.2 (A), R21.1
- new net: C28.2, R16.2
- new net +3.3VA: C19.1, C27.1, C30.1, R8.2, U3.13 (VDDA/VREF+)
- new net NRST: C22.1, J3.1 (Pin_1), SW1.3, SW1.4, U3.7 (NRST)
- new net OSC_IN: C23.1, U3.5 (PH0_OSC_IN), X1.1 (OSC1)
- new net OSC_OUT: R15.2, U3.6 (PH1_OSC_OUT)
- new net SWCLK: J3.3 (Pin_3), U3.49 (PA14)
- new net SWDIO: J3.2 (Pin_2), U3.46 (PA13)
- new net USART2_RX: J3.5 (Pin_5), U3.17 (PA3)
- new net USART2_TX: J3.6 (Pin_6), U3.16 (PA2)
- new net V_CAP: C29.1, U3.30 (VCAP_1)
- no-connect marks 9 -> 12
Other:
- note added: "Notes: -add Gyro pins in case the SMD does not work to use the module"
- note added: "Reverse polarity & overvoltage protection"
- note added: "all should be placed as close as possible, besides the RST btn"
- note added: "one as close as possible to each VDD pin"
- note added: "propgraming header"
- note added: "uC"
- note added: "uC minimal"
- note removed: "Notes: -change to BD9G101G and power the motors directly from the battery. No need for the 3A that i have now -design reverse polarity protection (order TVS(?) diode)"
- moved on the sheet: C3, C5, C6, C7, C8, C9, R1, R2

Commit message: pin assignments KiCad
Connections:
- net HC-05 STATE: now also U3.45 (PA12); no longer U3.41 (PA8)
- net USART1_RX: now also J3.5 (Pin_5)
- net USART1_TX: now also J3.6 (Pin_6)
- net USW2: now reaches U3.10 (PC2)
- net USW3: now reaches U3.11 (PC3)
- net ENC1_A: now reaches U3.14 (PA0)
- net ENC1_B: now reaches U3.15 (PA1)
- net UBTN1: now reaches U3.2 (PC13)
- net SENS3_ADC: now reaches U3.20 (PA4)
- net SESN4_ADC: now reaches U3.21 (PA5)
- net SENS5_ADC: now reaches U3.22 (PA6)
- net ULED1: now reaches U3.23 (PA7)
- net ULED2: now reaches U3.24 (PC4)
- net ULED3: now reaches U3.25 (PC5)
- net SENS3_PWM: now reaches U3.26 (PB0)
- net SENS4_PWM: now reaches U3.27 (PB1)
- net UBTN2: now reaches U3.3 (PC14-OSC32_IN)
- net M1A: now reaches U3.39 (PC8)
- net M1B: now reaches U3.40 (PC9)
- net M2_PWM: now reaches U3.44 (PA11)
- net ENC2_A: now reaches U3.50 (PA15)
- net M2A: now reaches U3.51 (PC10)
- net M2B: now reaches U3.52 (PC11)
- net MOTORS_EN: now reaches U3.53 (PC12)
- net ENC2_B: now reaches U3.55 (PB3)
- net SENS1_PWM: now reaches U3.56 (PB4)
- net SENS2_PWM: now reaches U3.57 (PB5)
- net EEPROM_SCL: now reaches U3.58 (PB6)
- net EEPROM_SDA: now reaches U3.59 (PB7)
- net EDF_PWM: now reaches U3.61 (PB8)
- net SENS5_PWM: now reaches U3.62 (PB9)
- net BAT_MON: now reaches U3.8 (PC0)
- net USW1: now reaches U3.9 (PC1)
- net SPI2_CS renamed GYRO_CS
- net SPI2_MISO renamed GYRO_MISO
- net SPI2_MOSI renamed GYRO_MOSI
- net SPI2_SCK renamed GYRO_SCK
- net SWCLK renamed TCK
- net SWDIO renamed TMS
- net USART2_RX renamed SENS2_ADC
- net SENS2_ADC: no longer J3.5 (Pin_5)
- net USART2_TX renamed SENS1_ADC
- net SENS1_ADC: no longer J3.6 (Pin_6)
- new net M1_PWM: U3.41 (PA8)
Other:
- moved on the sheet: R18, U3

Commit message: schematic add: UBTNS, USWS, ENC1,2, EEPROM, ULEDS
Parts:
- added C11, C37, C38, C39, C40: 100nF, LCSC:C_0805_2012Metric_Pad1.18x1.45mm_HandSolder, symbol Device:C
- added LED1: XL-2012SURC, LCSC:C965812_LED0805-RD_RED, symbol LCSC:XL-2012SURC
- added LED2: XL-2012UBC, LCSC:C965817_LED0805-RD, symbol LCSC:XL-2012UBC
- added LED3: XL-2012UGC, LCSC:C965815_LED0805-RD_GREEN, symbol LCSC:XL-2012UGC
- added R19: 100, LCSC:R_0805_2012Metric_Pad1.20x1.40mm_HandSolder, symbol Device:R
- added R20, R28, R29: 4.7k, LCSC:R_0805_2012Metric_Pad1.20x1.40mm_HandSolder, symbol Device:R
- added R22, R23, R24: 1k, LCSC:R_0805_2012Metric_Pad1.20x1.40mm_HandSolder, symbol Device:R
- added R25, R26, R27: ?k, LCSC:R_0805_2012Metric_Pad1.20x1.40mm_HandSolder, symbol Device:R
- added SW3: TS60110-411-03015, LCSC:C42400889_SW-SMD_4P-L5_2-W5_2-P3_70-LS6_4-BL, symbol LCSC:TS60110-411-03015
- added SW4, SW5, SW6: MST22D18G2 125, lcsc_footprints:C2906280_SW-SMD_MST22D18G2, symbol LCSC:MST22D18G2_125
- added U7: AT24C256C-SSHL-T, LCSC:C6482_SOIC-8_L4_9-W3_9-P1_27-LS6_0-BL, symbol LCSC:AT24C256C-SSHL-T
Connections:
- net +3V3: now also C11.2, R20.2, R28.1, R29.1, SW4.3, SW4.6, SW5.3, SW5.6, SW6.3, SW6.6, U7.8 (VCC)
- net EEPROM_SCL: now also R29.2, U7.6 (SCL)
- net EEPROM_SDA: now also R28.2, U7.5 (SDA)
- net ENC1_A: now also U2.6 (A)
- net ENC1_B: now also U2.7 (B)
- net ENC2_A: now also U6.6 (A)
- net ENC2_B: now also U6.7 (B)
- net GND: now also C11.1, C38.1, C39.1, C40.1, R19.1, R25.2, R26.2, R27.2, SW3.3, SW3.4, SW4.1, SW4.4, SW5.1, SW5.4, SW6.1, SW6.4, U7.1 (A0), U7.2 (A1), U7.3 (A2), U7.4 (GND), U7.7 (WP)
- net UBTN1: now also C28.1, R17.1, SW2.1, SW2.2
- net UBTN2: now also C37.1, R20.1, SW3.1, SW3.2
- net ULED1: now also LED1.2 (A)
- net ULED2: now also LED2.2 (A)
- net ULED3: now also LED3.2 (A)
- net USW1: now also R22.2, SW4.2, SW4.5
- net USW2: now also R23.2, SW5.2, SW5.5
- net USW3: now also R24.2, SW6.2, SW6.5
- new net: C40.2, R24.1
- new net: LED1.1 (K), R25.1
- new net: LED2.1 (K), R26.1
- new net: C37.2, R19.2
- new net: LED3.1 (K), R27.1
- new net: C38.2, R22.1
- new net: C39.2, R23.1
Other:
- note added: "EEPROM"
- note added: "Encoders"
- note added: "uC User"
- moved on the sheet: C1, C10, C13, C16, C18, C19, C2, C28, C3, C4, C5, C6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

Commit message: bat monitor + EDF
Parts:
- added C12: 10uF, LCSC:C_0805_2012Metric_Pad1.18x1.45mm_HandSolder, symbol Device:C
- added C14: 330nF, LCSC:C_0805_2012Metric_Pad1.18x1.45mm_HandSolder, symbol Device:C
- added C15: 100pF, LCSC:C_0805_2012Metric_Pad1.18x1.45mm_HandSolder, symbol Device:C
- added C17, C20: 22uF, LCSC:C_0805_2012Metric_Pad1.18x1.45mm_HandSolder, symbol Device:C
- added C21: 100nF, LCSC:C_0805_2012Metric_Pad1.18x1.45mm_HandSolder, symbol Device:C
- added D5, D6: SS26-LTP, LCSC:C85690_SMA_L4_3-W2_6-LS5_2-RD, symbol LCSC:SS26-LTP
- added J4: Conn_01x02_Pin, Connector_PinHeader_2.54mm:PinHeader_1x02_P2.54mm_Vertical, symbol Connector:Conn_01x02_Pin
- added L2: APH0420T3R3M, LCSC:C5349667_IND-SMD_L4_4-W4_2, symbol LCSC:APH0420T3R3M
- added Q1: AO3400A, LCSC:C20917_SOT-23-3_L2_9-W1_3-P1_90-LS2_4-BR, symbol LCSC:AO3400A
- added R3: 31.6k, LCSC:R_0805_2012Metric_Pad1.20x1.40mm_HandSolder, symbol Device:R
- added R30: 100, LCSC:R_0805_2012Metric_Pad1.20x1.40mm_HandSolder, symbol Device:R
- added R31, R4: 10k, LCSC:R_0805_2012Metric_Pad1.20x1.40mm_HandSolder, symbol Device:R
- added R32: /DNP, LCSC:R_0805_2012Metric_Pad1.20x1.40mm_HandSolder, symbol Device:R
- added R33, R34: ?k, LCSC:R_0805_2012Metric_Pad1.20x1.40mm_HandSolder, symbol Device:R
- added U8: AP62300Z6-7, LCSC:C5250745_SOT-563-6_L1_6-W1_2-P0_50-LS1_6-BL, symbol LCSC:AP62300Z6-7
Connections:
- net +5V: now also U8.5 (EN)
- net +BATT: now also C12.1, R32.1, R33.2, U8.1 (VIN)
- net BAT_MON: now also C21.1, R33.1, R34.2
- net EDF_PWM: now also R30.1
- net GND: now also C12.2, C17.2, C20.2, C21.2, Q1.2 (S), R31.2, R34.1, R4.2, U8.3 (GND)
- new net: C15.2, R3.2, R4.1, U8.6 (FB)
- new net: C14.2, L2.1, U8.2 (SW)
- new net: D5.2 (A), D6.2 (A), J4.2 (Pin_2), Q1.3 (D)
- new net: C14.1, U8.4 (BST)
- new net: Q1.1 (G), R30.2, R31.1
- new net V_EDF: C15.1, C17.1, C20.1, D5.1 (C), D6.1 (C), J4.1 (Pin_1), L2.2, R3.1, R32.2
Other:
- note added: "3v3 config change resistors for bigger voltage Option for bypass"
- note added: "Bat monitor"
- note added: "EDF"
- moved on the sheet: J3

Commit message: added encoders connectors
Parts:
- removed C11: 100nF, LCSC:C_0805_2012Metric_Pad1.18x1.45mm_HandSolder, symbol Device:C
- removed R28, R29: 4.7k, LCSC:R_0805_2012Metric_Pad1.20x1.40mm_HandSolder, symbol Device:R
- removed U7: AT24C256C-SSHL-T, LCSC:C6482_SOIC-8_L4_9-W3_9-P1_27-LS6_0-BL, symbol LCSC:AT24C256C-SSHL-T
- added C41: 100nF, LCSC:C_0805_2012Metric_Pad1.18x1.45mm_HandSolder, symbol Device:C
- added J5, J6: Conn_01x04_Socket, Connector_PinSocket_2.54mm:PinSocket_1x04_P2.54mm_Vertical, symbol Connector:Conn_01x04_Socket
- added J7, J8: Conn_01x04_Pin, Connector_PinSocket_2.54mm:PinSocket_1x04_P2.54mm_Vertical, symbol Connector:Conn_01x04_Pin
- added R35, R36: 4.7k, LCSC:R_0805_2012Metric_Pad1.20x1.40mm_HandSolder, symbol Device:R
- added U9: AT24C256C-SSHL-T, LCSC:C6482_SOIC-8_L4_9-W3_9-P1_27-LS6_0-BL, symbol LCSC:AT24C256C-SSHL-T
Connections:
- net +3V3: now also C41.2, J5.1 (Pin_1), J6.1 (Pin_1), R35.1, R36.1, U9.8 (VCC); no longer C10.1, C3.1, D1.1 (K), D4.1 (K), U2.1 (VDD), U6.1 (VDD)
- net EEPROM_SCL: now also R36.2, U9.6 (SCL)
- net EEPROM_SDA: now also R35.2, U9.5 (SDA)
- net ENC1_A: now also J5.3 (Pin_3); no longer U2.6 (A)
- net ENC1_B: now also J5.2 (Pin_2); no longer U2.7 (B)
- net ENC2_A: now also J6.3 (Pin_3); no longer U6.6 (A)
- net ENC2_B: now also J6.2 (Pin_2); no longer U6.7 (B)
- net GND: now also C41.1, J5.4 (Pin_4), J6.4 (Pin_4), U9.1 (A0), U9.2 (A1), U9.3 (A2), U9.4 (GND), U9.7 (WP); no longer C10.2, C3.2, D1.2 (A), D4.2 (A), U2.2 (MODE), U2.4 (GND), U6.2 (MODE), U6.4 (GND)
- new net 3v3_BRD: C10.1, C3.1, D1.1 (K), D4.1 (K), J7.1 (Pin_1), J8.1 (Pin_1), U2.1 (VDD), U6.1 (VDD)
- new net ENC1_A_BRD: J7.3 (Pin_3)
- new net ENC1_B_BRD: J7.2 (Pin_2)
- new net ENC2_A_BRD: J8.3 (Pin_3), U6.6 (A)
- new net ENC2_B_BRD: J8.2 (Pin_2), U6.7 (B)
- new net GND_BRD: C10.2, C3.2, D1.2 (A), D4.2 (A), J7.4 (Pin_4), J8.4 (Pin_4), U2.2 (MODE), U2.4 (GND), U6.2 (MODE), U6.4 (GND)
Other:
- note added: "Encoder connectors"
- note added: "Notes: -add Gyro pins in case the SMD does not work to use the module -add encoders pins - encoder circuit will be homemade as it is simple"
- note removed: "Notes: -add Gyro pins in case the SMD does not work to use the module"

Commit message: footprint update
Parts:
- SW4, SW5, SW6: footprint lcsc_footprints:C2906280_SW-SMD_MST22D18G2 -> LCSC:C2906280_SW-SMD_MST22D18G2
Changed lines of the file:
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@@
 		(fields_autoplaced yes)
 		(property "Reference" "SW6"
-			(at 108.585 155.5749 0)
+			(at 109.22 155.5749 0)
 			(show_name no)
 			(do_not_autoplace no)
@@
 		)
 		(property "Value" "MST22D18G2 125"
-			(at 108.585 158.1149 0)
+			(at 109.22 158.1149 0)
 			(show_name no)
 			(do_not_autoplace no)
@@
 			)
 		)
-		(property "Footprint" "lcsc_footprints:C2906280_SW-SMD_MST22D18G2"
+		(property "Footprint" "LCSC:C2906280_SW-SMD_MST22D18G2"
 			(at 100.965 167.005 0)
 			(hide yes)
@@
 			)
 		)
-		(property "Footprint" "lcsc_footprints:C2906280_SW-SMD_MST22D18G2"
+		(property "Footprint" "LCSC:C2906280_SW-SMD_MST22D18G2"
 			(at 34.29 167.005 0)
 			(hide yes)
@@
 			)
 		)
-		(property "Footprint" "lcsc_footprints:C2906280_SW-SMD_MST22D18G2"
+		(property "Footprint" "LCSC:C2906280_SW-SMD_MST22D18G2"
 			(at 68.58 167.005 0)
 			(hide yes)
