File: KiCad/PCB_V1/PCB_V1.kicad_sch (KiCad schematic)
At the start: 101 parts, among them J1 Conn_01x06_Socket, J2 Conn_01x02_Pin, J3 Conn_01x07_Pin, J4 Conn_01x02_Pin, J5 Conn_01x04_Socket, J6 Conn_01x04_Socket, J7 Conn_01x04_Pin, J8 Conn_01x04_Pin, Q1 AO3400A, SW1 TS60110-411-03015, SW2 TS60110-411-03015, SW3 TS60110-411-03015, SW4 MST22D18G2 125, SW5 MST22D18G2 125, SW6 MST22D18G2 125, U1 LSM6DSOXTR, U2 MT6701CT-ACD_C50203010, U3 STM32F411RET6, U4 AP62300Z6-7, U5 TLV75533PDBVR, U6 MT6701CT-ACD_C50203010, U8 AP62300Z6-7, U9 AT24C256C-SSHL-T, X1 X49SS2-8.000-F20JGDT

Commit message: motor drv + gyro connector schematic
Parts:
- removed C4: 100nF, LCSC:C_0805_2012Metric_Pad1.18x1.45mm_HandSolder, symbol Device:C
- added C11, C42, C44: 100nF, LCSC:C_0805_2012Metric_Pad1.18x1.45mm_HandSolder, symbol Device:C
- added C43, C45: 10uF, LCSC:C_0805_2012Metric_Pad1.18x1.45mm_HandSolder, symbol Device:C
- added J10, J9: Conn_01x02_Pin, Connector_PinHeader_2.54mm:PinHeader_1x02_P2.54mm_Vertical, symbol Connector:Conn_01x02_Pin
- added J11: Conn_01x06_Socket, Connector_PinSocket_2.54mm:PinSocket_1x06_P2.54mm_Vertical, symbol Connector:Conn_01x06_Socket
- added R5: 10k, LCSC:R_0805_2012Metric_Pad1.20x1.40mm_HandSolder, symbol Device:R
- added U7: TB6612FNG,C,8,EL, LCSC:C141517_SSOP-24_L8_3-W5_6-P0_65-LS7_6-BL, symbol LCSC:TB6612FNG,C,8,EL
Connections:
- net +3V3: now also J1.6 (Pin_6), C11.2, C42.2, C43.2, J11.5 (Pin_5), U7.20 (VCC); no longer J1.5 (Pin_5)
- net +BATT: now also C44.2, C45.2, U7.13 (VM2), U7.14 (VM3), U7.24 (VM1)
- net GND: now also J1.5 (Pin_5), C11.1, C42.1, C43.1, C44.1, C45.1, J11.4 (Pin_4), R5.2, U7.10 (PGND2), U7.18 (GND), U7.3 (PGND1), U7.4 (PGND1), U7.9 (PGND2); no longer J1.4 (Pin_4)
- net GYRO_CS: now also J1.4 (Pin_4)
- net GYRO_MISO: now also J1.2 (Pin_2)
- net GYRO_MOSI: now also J1.1 (Pin_1)
- net GYRO_SCK: now also J1.3 (Pin_3)
- net HC-05 STATE: now also J11.1 (Pin_1); no longer J1.1 (Pin_1)
- net M1A: now also U7.21 (AIN1)
- net M1B: now also U7.22 (AIN2)
- net M1_PWM: now also U7.23 (PWMA)
- net M2A: now also U7.17 (BIN1)
- net M2B: now also U7.16 (BIN2)
- net M2_PWM: now also U7.15 (PWMB)
- net MOTORS_EN: now also R5.1, U7.19 (STBY)
- net USART1_RX: now also J11.3 (Pin_3); no longer J1.3 (Pin_3)
- net USART1_TX: now also J11.2 (Pin_2); no longer J1.2 (Pin_2)
- new net: J9.1 (Pin_1), U7.1 (AO1), U7.2 (AO1)
- new net: J9.2 (Pin_2), U7.5 (AO2), U7.6 (AO2)
- new net: J10.1 (Pin_1), U7.7 (BO2), U7.8 (BO2)
- new net: J10.2 (Pin_2), U7.11 (BO1), U7.12 (BO1)
Other:
- note added: "Gyro connector"
- note added: "Motor driver"
- note added: "if necessary in case SMD does not work"
